File: PCB/hackpad.kicad_sch (KiCad schematic)
At the start: 12 parts, among them J1 Conn_01x04_Pin, SW1 SW_Push, SW2 SW_Push, SW3 SW_Push, SW4 SW_Push, SW5 SW_Push, SW6 RotaryEncoder_Switch, U1 XIAO-RP2040-DIP

Commit message: updates from the last 4 days
mostly 3d models for cad stuff and kicad mod..?
Parts:
- added D5: SK6812MINI, Custom:MX_SK6812MINI-E_REV(1), symbol LED:SK6812MINI
- D1, D2, D3, D4: footprint LED_SMD:LED_SK6812MINI_PLCC4_3.5x3.5mm_P1.75mm -> Custom:MX_SK6812MINI-E_REV(1)
- SW1, SW2, SW3, SW4, SW5: footprint Button_Switch_Keyboard:SW_Cherry_MX_1.00u_PCB -> Custom:cherry_mx_1.00u_pcb_custom
- SW6: footprint Rotary_Encoder:RotaryEncoder_Alps_EC11E-Switch_Vertical_H20mm -> Custom:Rotary_EncoderRotaryEncoder_Alps_EC11E-Switch_Vertical_H20mm_custom
Connections:
- net +5V: now also D5.4 (VDD)
- net GND: now also D5.2 (VSS)
- net at D4.1 (DOUT): now also D5.3 (DIN)
Changed lines of the file:
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@@
+	)
+	(junction
+		(at 175.26 35.56)
+		(diameter 0)
+		(color 0 0 0 0)
 	)
 	(junction
@@
 		(color 0 0 0 0)
 	)
+	(junction
+		(at 175.26 50.8)
+		(diameter 0)
+		(color 0 0 0 0)
+	)
 	(wire
 		(pts
@@
 	(wire
 		(pts
-			(xy 134.62 35.56) (xy 144.78 35.56)
+			(xy 175.26 35.56) (xy 195.58 35.56)
 		)
 		(stroke
@@
 	(wire
 		(pts
-			(xy 134.62 50.8) (xy 144.78 50.8)
+			(xy 134.62 35.56) (xy 144.78 35.56)
 		)
 		(stroke
@@
 	(wire
 		(pts
-			(xy 114.3 35.56) (xy 134.62 35.56)
+			(xy 134.62 50.8) (xy 144.78 50.8)
 		)
 		(stroke
@@
 	(wire
 		(pts
-			(xy 114.3 50.8) (xy 134.62 50.8)
+			(xy 114.3 35.56) (xy 134.62 35.56)
 		)
 		(stroke
@@
 	(wire
 		(pts
-			(xy 162.56 43.18) (xy 167.64 43.18)
+			(xy 175.26 50.8) (xy 195.58 50.8)
 		)
 		(stroke
@@
 	(wire
 		(pts
-			(xy 144.78 35.56) (xy 154.94 35.56)
+			(xy 114.3 50.8) (xy 134.62 50.8)
 		)
 		(stroke
@@
 	(wire
 		(pts
-			(xy 154.94 35.56) (xy 175.26 35.56)
+			(xy 162.56 43.18) (xy 167.64 43.18)
 		)
 		(stroke
@@
 		)
 	)
+	(wire
+		(pts
+			(xy 182.88 43.18) (xy 187.96 43.18)
+		)
+		(stroke
+			(width 0)
+			(type default)
+		)
+	)
+	(wire
+		(pts
+			(xy 144.78 35.56) (xy 154.94 35.56)
+		)
+		(stroke
+			(width 0)
+			(type default)
+		)
+	)
+	(wire
+		(pts
+			(xy 154.94 35.56) (xy 175.26 35.56)
+		)
+		(stroke
+			(width 0)
+			(type default)
+		)
+	)
 	(global_label "Button 3"
 		(shape input)
@@
 			)
 		)
-		(property "Footprint" "Rotary_Encoder:RotaryEncoder_Alps_EC11E-Switch_Vertical_H20mm"
+		(property "Footprint" "Custom:Rotary_EncoderRotaryEncoder_Alps_EC11E-Switch_Vertical_H20mm_custom"
 			(at 229.87 139.446 0)
 			(effects
@@
 			)
 		)
-		(property "Footprint" "Button_Switch_Keyboard:SW_Cherry_MX_1.00u_PCB"
+		(property "Footprint" "Custom:cherry_mx_1.00u_pcb_custom"
 			(at 233.68 123.19 0)
 			(effects
@@
 			)
 		)
-		(property "Footprint" "Button_Switch_Keyboard:SW_Cherry_MX_1.00u_PCB"
+		(property "Footprint" "Custom:cherry_mx_1.00u_pcb_custom"
 			(at 233.68 69.85 0)
 			(effects
@@
 			)
 		)
-		(property "Footprint" "Button_Switch_Keyboard:SW_Cherry_MX_1.00u_PCB"
+		(property "Footprint" "Custom:cherry_mx_1.00u_pcb_custom"
 			(at 233.68 110.49 0)
 			(effects
@@
 			)
 		)
-		(property "Footprint" "Button_Switch_Keyboard:SW_Cherry_MX_1.00u_PCB"
+		(property "Footprint" "Custom:cherry_mx_1.00u_pcb_custom"
 			(at 233.68 83.82 0)
 			(effects
@@
 			)
 		)
-		(property "Footprint" "Button_Switch_Keyboard:SW_Cherry_MX_1.00u_PCB"
+		(property "Footprint" "Custom:cherry_mx_1.00u_pcb_custom"
 			(at 233.68 97.79 0)
 			(effects
@@
 			)
 		)
-		(property "Footprint" "LED_SMD:LED_SK6812MINI_PLCC4_3.5x3.5mm_P1.75mm"
+		(property "Footprint" "Custom:MX_SK6812MINI-E_REV(1)"
 			(at 176.53 50.8 0)
 			(effects
@@
 			)
 		)
-		(property "Footprint" "LED_SMD:LED_SK6812MINI_PLCC4_3.5x3.5mm_P1.75mm"
+		(property "Footprint" "Custom:MX_SK6812MINI-E_REV(1)"
 			(at 115.57 50.8 0)
 			(effects
@@
 	(symbol
 		(lib_id "LED:SK6812MINI")
+		(at 195.58 43.18 0)
+		(unit 1)
+		(exclude_from_sim no)
+		(in_bom yes)
+		(on_board yes)
+		(dnp no)
+		(fields_autoplaced yes)
+		(property "Reference" "D5"
+			(at 208.28 36.7598 0)
+			(effects
+				(font
+					(size 1.27 1.27)
+				)
+				(hide yes)
+			)
+		)
+		(property "Value" "SK6812MINI"
+			(at 208.28 39.2998 0)
+			(effects
+				(font
+					(size 1.27 1.27)
+				)
+				(hide yes)
+			)
+		)
+		(property "Footprint" "Custom:MX_SK6812MINI-E_REV(1)"
+			(at 196.85 50.8 0)
+			(effects
+				(font
+					(size 1.27 1.27)
+				)
+				(justify left top)
+				(hide yes)
+			)
+		)
+		(property "Datasheet" "https://cdn-shop.adafruit.com/product-files/2686/SK6812MINI_REV.01-1-2.pdf"
+			(at 198.12 52.705 0)
+			(effects
+				(font
+					(size 1.27 1.27)
+				)
+				(justify left top)
+				(hide yes)
+			)
+		)
+		(property "Description" "RGB LED with integrated controller"
+			(at 195.58 43.18 0)
+			(effects
+				(font
+					(size 1.27 1.27)
+				)
+				(hide yes)
+			)
+		)
+		(pin "1"
+		)
+		(pin "4"
+		)
+		(pin "3"
+		)
+		(pin "2"
+		)
+		(instances
+			(project "hackpad"
+				(path "/3efa313a-c978-4e87-bae9-dd1e3a1b5bbc"
+					(reference "D5")
+					(unit 1)
+				)
+			)
+		)
+	)
+	(symbol
+		(lib_id "LED:SK6812MINI")
 		(at 154.94 43.18 0)
 		(unit 1)
@@
 			)
 		)
-		(property "Footprint" "LED_SMD:LED_SK6812MINI_PLCC4_3.5x3.5mm_P1.75mm"
+		(property "Footprint" "Custom:MX_SK6812MINI-E_REV(1)"
 			(at 156.21 50.8 0)
 			(effects
@@
 			)
 		)
-		(property "Footprint" "LED_SMD:LED_SK6812MINI_PLCC4_3.5x3.5mm_P1.75mm"
+		(property "Footprint" "Custom:MX_SK6812MINI-E_REV(1)"
 			(at 135.89 50.8 0)
 			(effects
